Commit message: Finished

File: checkpoint8_auxiliary_files/rb1_ros2_description/xacro/rb1_ros2_base.urdf.xacro (robot description, xacro)
@@ -126,4 +126,13 @@
         <state_interface name="effort"/>
       </joint>
+      <joint name="$(arg prefix)elevator_platform_joint">
+              <command_interface name="effort">
+        <param name="min">-10</param>
+        <param name="max">10</param>
+      </command_interface>
+      <state_interface name="position"/>
+      <state_interface name="velocity"/>
+      <state_interface name="effort"/>
+    </joint>
     </ros2_control>
 </robot>
